Commit message: add: odom link.

File: motor_node/xacro/robot.xacro (robot description, xacro)
@@ -1,4 +1,4 @@
 <?xml version="1.0"?>
-<robot name="dtw_robot" xmlns:xacro="http://ros.org/wiki/xacro">
+<robot name="robot" xmlns:xacro="http://ros.org/wiki/xacro">
   <material name="gray">
     <color rgba="0.5 0.5 0.5 2.5"/>
@@ -26,5 +26,10 @@
     </link>
   </xacro:macro>
+  <link name="odom"/>
   <link name="base_link"/>
+  <joint name="base_joint" type="floating">
+    <parent link="odom"/>
+    <child  link="base_link"/>
+  </joint>
   <joint name="body_joint_up" type="fixed">
     <parent link="base_link"/>
