Commit message: add: ZED urdf.

File: motor_node/xacro/roombot.xacro (robot description, xacro)
@@ -31,4 +31,5 @@
     <parent link="odom"/>
     <child  link="base_link"/>
+    <origin xyz="0 0 0" rpy="0 0 0"/>
   </joint>
   <joint name="body_joint_up" type="fixed">
@@ -76,18 +77,4 @@
    </visual>
   </link>
-  <joint name="zed_joint" type="fixed">
-    <parent link="body_link_up" />
-    <child link="zed_link" />
-    <origin xyz="0.068 -0.01 0.017 " rpy="0 0 0" />
-  </joint>
-  <link name="zed_link">
-    <visual>
-      <geometry>
-        <mesh filename="package://zed_wrapper/urdf/models/ZEDM.stl" />
-      </geometry>
-      <origin xyz="0 0 0 " rpy="0 0 0" />
-      <material name="dark_gray" />
-    </visual>
-  </link>
   <joint name="rplidar_joint" type="fixed">
     <parent link="body_link_up" />
@@ -118,3 +105,54 @@
     </visual>
   </link>
+  <!-- ZED mini -->
+  <!-- Camera Center -->
+  <joint name="zed_camera_center_joint" type="fixed">
+    <parent link="body_link_up" />
+    <child link="zed_camera_center"/>
+    <origin xyz="0.068 -0.01 0.017 " rpy="0 0 0" />
+  </joint>
+  <link name="zed_camera_center">
+    <visual>
+      <origin xyz="0 0 0" rpy="0 0 0"/>
+      <geometry>
+        <mesh filename="package://zed_wrapper/urdf/models/ZEDM.stl" />
+      </geometry>
+      <material name="light_grey">
+        <color rgba="0 0 0 0.9"/>
+      </material>
+    </visual>
+  </link>
+  <!-- Left Camera -->
+  <joint name="zed_left_camera_joint" type="fixed">
+    <parent link="zed_camera_center"/>
+    <child link="zed_left_camera_frame"/>
+    <origin xyz="0 0.03 0" rpy="0 0 0" />
+  </joint>
+  <link name="zed_left_camera_frame" />
+  <joint name="zed_left_camera_optical_joint" type="fixed">
+    <origin xyz="0 0 0" rpy="-1.57079632679 0.0 -1.57079632679"/>
+    <parent link="zed_left_camera_frame"/>
+    <child link="zed_left_camera_optical_frame"/>
+  </joint>
+  <link name="zed_left_camera_optical_frame"/>
+  <!-- Right Camera -->
+  <joint name="zed_right_camera_joint" type="fixed">
+    <parent link="zed_camera_center"/>
+    <child link="zed_right_camera_frame"/>
+    <origin xyz="0 -0.03 0" rpy="0 0 0" />
+  </joint>
+  <link name="zed_right_camera_frame" />
+  <joint name="zed_right_camera_optical_joint" type="fixed">
+    <origin xyz="0 0 0" rpy="-1.57079632679 0.0 -1.57079632679"/>
+    <parent link="zed_right_camera_frame"/>
+    <child link="zed_right_camera_optical_frame"/>
+  </joint>
+  <link name="zed_right_camera_optical_frame"/>
+  <!-- IMU -->
+  <joint name="imu_link_joint" type="floating">
+    <parent link="zed_camera_center"/>
+    <child link="zed_imu_link"/>
+    <origin xyz="0 0 0" rpy="0 0 0" />
+  </joint>
+  <link name="zed_imu_link" />
 </robot>
